Commit message: skid steer controller

File: pluto_description/urdf/pluto.urdf.xacro (robot description, xacro)
@@ -8,5 +8,5 @@
   <xacro:include filename="$(find uos_common_urdf)/common.xacro" />
   <xacro:include filename="$(find uos_common_urdf)/urdf/imu.gazebo.urdf.xacro" />
-  <xacro:include filename="$(find riegl_driver)/urdf/riegl_vz400i_mount.urdf.xacro" />
+  <!--xacro:include filename="$(find riegl_driver)/urdf/riegl_vz400i_mount.urdf.xacro" /-->
   <xacro:property name="M_PI" value="3.14159265359"/>
   <xacro:property name="footprint_to_base_rpy_p" value="-0.142"/>
@@ -58,5 +58,4 @@
     value="${body_height/2 -(vertical_lever_height + 0.03
       - bearing_width/2)}"/>
-  <xacro:property name="wheel_radius" value="0.103" />
   <xacro:property name="axis_length" value="0.47" />
   <xacro:property name="turning_adaptation" value="0.95" />
@@ -90,4 +89,7 @@
         <mesh filename="package://pluto_description/meshes/pluto_base_collision.stl"/>
       </geometry>
+      <material name="silver" >
+        <color rgba="0.5 0.5 0.5 1" />
+      </material>
     </collision>
     <xacro:box_inertial
@@ -103,4 +105,7 @@
     <child link="base_link" />
   </joint>
+  <gazebo reference="base_link">
+    <material>Gazebo/Grey</material>
+  </gazebo>
   <!--Virtual Axis Macro-->
   <xacro:macro name="virtual_axis" params="side xyz rot">
@@ -271,5 +276,5 @@
   </joint>
   <!-- inertial measurement unit for gazebo -->
-  <xacro:imu_gazebo link="imu" imu_topic="imu/data" update_rate="100.0" stdev="${imu_stdev}" />
+  <xacro:imu_gazebo link="imu_center" imu_topic="imu/data" update_rate="100.0" stdev="${imu_stdev}" />
   <link name="velodyne">
     <visual>
@@ -292,5 +297,5 @@
       rpy="0 0 0" />
   </joint>
-  <joint name="riegl_vz400i_to_base_joint" type="fixed">
+  <!--joint name="riegl_vz400i_to_base_joint" type="fixed">
     <child link="riegl_mount_base" />
     <parent link="base_link" />
@@ -300,5 +305,5 @@
             ${riegl_vz400i_offset_z}"
       rpy="0 0 0" />
-  </joint>
+  </joint-->
   <!-- GPS Sensor -->
   <gazebo reference="velodyne">
@@ -349,23 +354,19 @@
       <velocityGaussianNoise>0.1 0.1 0.1</velocityGaussianNoise>
     </plugin>
-   </gazebo>
+  </gazebo>
   <gazebo>
-    <plugin name="volksbot_diffdrive" filename="libgazebo_ros_diffdrive_uos.so">
-      <alwaysOn>true</alwaysOn>
-      <cmd_vel_topic_name>cmd_vel</cmd_vel_topic_name>
-      <odom_topic_name>odom</odom_topic_name>
-      <joint_states_topic_name>joint_states</joint_states_topic_name>
-      <left_front_wheel_joint>left_front_wheel_joint</left_front_wheel_joint>
-      <left_middle_wheel_joint>left_middle_wheel_joint</left_middle_wheel_joint>
-      <left_rear_wheel_joint>left_rear_wheel_joint</left_rear_wheel_joint>
-      <right_front_wheel_joint>right_front_wheel_joint</right_front_wheel_joint>
-      <right_middle_wheel_joint>right_middle_wheel_joint</right_middle_wheel_joint>
-      <right_rear_wheel_joint>right_rear_wheel_joint</right_rear_wheel_joint>
-      <wheel_separation>${axis_length}</wheel_separation>
-      <wheel_diameter>${2*wheel_radius}</wheel_diameter>
-      <turning_adaptation>${turning_adaptation}</turning_adaptation>
-      <torque>4.0</torque>
-      <max_velocity>1.0</max_velocity>
-      <updateRate>40.0</updateRate>
+    <plugin name="skid_steer_drive_controller" filename="libgazebo_ros_skid_steer_drive.so">
+      <updateRate>100.0</updateRate>
+      <robotNamespace>/</robotNamespace>
+      <leftFrontJoint>left_front_wheel_joint</leftFrontJoint>
+      <rightFrontJoint>right_front_wheel_joint</rightFrontJoint>
+      <leftRearJoint>left_rear_wheel_joint</leftRearJoint>
+      <rightRearJoint>right_rear_wheel_joint</rightRearJoint>
+      <wheelSeparation>${axis_length}</wheelSeparation>
+      <wheelDiameter>${2*wheel_radius}</wheelDiameter>
+      <robotBaseFrame>base_link</robotBaseFrame>
+      <torque>20</torque>
+      <topicName>cmd_vel</topicName>
+      <broadcastTF>false</broadcastTF>
     </plugin>
   </gazebo>

Commit message: fake gazebo localization

File: pluto_description/urdf/pluto.urdf.xacro (robot description, xacro)
@@ -169,6 +169,5 @@
         <origin xyz="0 0 0" rpy="0 0 0" />
         <geometry>
-          <mesh
-          filename="package://pluto_description/meshes/pluto_wheel_collision.stl"/>
+          <mesh filename="package://pluto_description/meshes/pluto_wheel.stl"/>
         </geometry>
       </collision>
@@ -185,9 +184,9 @@
     </joint>
     <gazebo reference="${name}_link">
-      <mu1>1</mu1>
-      <mu2>1</mu2>
+      <mu1>0.7</mu1>
+      <mu2>0.7</mu2>
       <material>Gazebo/Black</material>
-      <kp>10000000</kp>
-      <kd>10</kd>
+      <kp>10000000.0</kp>
+      <kd>1.0</kd>
       <selfCollide>false</selfCollide>
     </gazebo>
@@ -377,6 +376,6 @@
       <updateRate>30.0</updateRate>
       <bodyName>base_footprint</bodyName>
-      <topicName>base_footprint_pose_ground_truth</topicName>
-      <gaussianNoise>0.0</gaussianNoise>
+      <topicName>gazebo_odom</topicName>
+      <gaussianNoise>0.01</gaussianNoise>
       <frameName>map</frameName>
       <interface:position name="base_footprint_p3d_position_iface" />

Commit message: using diff_drive_controller gazebo plugin with ros control

File: pluto_description/urdf/pluto.urdf.xacro (robot description, xacro)
@@ -1,12 +1,12 @@
 <?xml version="1.0"?>
-<robot
-  xmlns:xacro="http://ros.org/wiki/xacro"
-  xmlns:controller="http://playerstage.sourceforge.net/gazebo/xmlschema/#controller"
-  xmlns:interface="http://playerstage.sourceforge.net/gazebo/xmlschema/#interface"
-  xmlns:sensor="http://playerstage.sourceforge.net/gazebo/xmlschema/#sensor"
-  name="pluto">
+<robot xmlns:xacro="http://ros.org/wiki/xacro"
+       xmlns:controller="http://playerstage.sourceforge.net/gazebo/xmlschema/#controller"
+       xmlns:interface="http://playerstage.sourceforge.net/gazebo/xmlschema/#interface"
+       xmlns:sensor="http://playerstage.sourceforge.net/gazebo/xmlschema/#sensor"
+       name="pluto">
   <xacro:include filename="$(find uos_common_urdf)/common.xacro" />
   <xacro:include filename="$(find uos_common_urdf)/urdf/imu.gazebo.urdf.xacro" />
   <!--xacro:include filename="$(find riegl_driver)/urdf/riegl_vz400i_mount.urdf.xacro" /-->
+  <xacro:include filename="$(find pluto_description)/urdf/wheel.urdf.xacro" />
   <xacro:property name="M_PI" value="3.14159265359"/>
   <xacro:property name="footprint_to_base_rpy_p" value="-0.142"/>
@@ -62,5 +62,5 @@
   <xacro:property name="body_mass" value="40.0"/>
   <xacro:property name="wheel_mass" value="3.0"/>
-  <xacro:property name="wheel_radius" value="0.15"/>
+  <xacro:property name="wheel_radius" value="0.103"/>
   <xacro:property name="wheel_thickness" value="0.065"/>
   <xacro:property name="imu_center_offset_x" value="${body_length/2 - 0.285}"/>
@@ -82,4 +82,8 @@
       <material name="silver" >
         <color rgba="0.5 0.5 0.5 1" />
+        <ambient>0.5 0.5 0.5 1</ambient>
+        <diffuse>0.5 0.5 0.5 1</diffuse>
+        <specular>0 0 0 0</specular>
+        <emissive>0 0 0 1</emissive>
       </material>
     </visual>
@@ -89,7 +93,4 @@
         <mesh filename="package://pluto_description/meshes/pluto_base_collision.stl"/>
       </geometry>
-      <material name="silver" >
-        <color rgba="0.5 0.5 0.5 1" />
-      </material>
     </collision>
     <xacro:box_inertial
@@ -99,4 +100,7 @@
       mass="${body_mass}"/>
   </link>
+  <gazebo reference="base_link">
+    <material>Gazebo/GreyTransparent</material>
+  </gazebo>
   <joint name="base_footprint_to_base_joint" type="fixed">
     <!-- origin xyz="0 0 0.2" rpy="0 ${-M_PI/18.0} 0" /-->
@@ -105,7 +109,4 @@
     <child link="base_link" />
   </joint>
-  <gazebo reference="base_link">
-    <material>Gazebo/Grey</material>
-  </gazebo>
   <!--Virtual Axis Macro-->
   <xacro:macro name="virtual_axis" params="side xyz rot">
@@ -132,4 +133,7 @@
         mass="${horizontal_lever_mass}"/>
     </link>
+    <gazebo reference="virtual_axis_${side}">
+      <material>Gazebo/GreyTransparent</material>
+    </gazebo>
     <joint name="virtual_${side}_to_base_joint" type="revolute">
       <origin xyz="${xyz}"
@@ -154,66 +158,22 @@
           ${virtual_axis_right_offset_z}"
     rot="0"/>
-  <!--Wheel Macro-->
-  <xacro:macro name="wheel" params="name parent xyz">
-    <link name="${name}_link">
-      <visual>
-        <origin xyz="0 0 0" rpy="0 0 0" />
-        <geometry>
-          <mesh filename="package://pluto_description/meshes/pluto_wheel.stl"/>
-        </geometry>
-        <material name="black" >
-          <color rgba="0 0 0 1" />
-        </material>
-      </visual>
-      <collision>
-        <origin xyz="0 0 0" rpy="0 0 0" />
-        <geometry>
-          <mesh filename="package://pluto_description/meshes/pluto_wheel.stl"/>
-        </geometry>
-      </collision>
-      <xacro:cylinder_inertial
-        radius="${wheel_radius}"
-        length="${wheel_thickness}"
-        mass="${wheel_mass}" />
-    </link>
-    <joint name="${name}_joint" type="continuous">
-      <origin xyz="${xyz}" rpy="0 0 0"/>
-      <parent link="${parent}"/>
-      <child link="${name}_link"/>
-      <axis xyz="0 1 0"/>
-    </joint>
-    <gazebo reference="${name}_link">
-      <mu1>0.7</mu1>
-      <mu2>0.7</mu2>
-      <material>Gazebo/Black</material>
-      <kp>10000000.0</kp>
-      <kd>1.0</kd>
-      <selfCollide>false</selfCollide>
-    </gazebo>
-  </xacro:macro>
-  <xacro:wheel
-    name="left_front_wheel"
-    parent="virtual_axis_left"
-    xyz="0.1075 0.095 0" />
-  <xacro:wheel
-    name="left_middle_wheel"
-    parent="virtual_axis_left"
-    xyz="-0.1075 0.095 0" />
-  <xacro:wheel
-    name="left_rear_wheel"
-    parent="base_link"
-    xyz="-0.23 0.19 ${(-body_height/2.0)+(bearing_height/2.0)}" />
-  <xacro:wheel
-    name="right_front_wheel"
-    parent="virtual_axis_right"
-    xyz="0.1075 -0.095 0" />
-  <xacro:wheel
-    name="right_middle_wheel"
-    parent="virtual_axis_right"
-    xyz="-0.1075 -0.095 0" />
-  <xacro:wheel
-    name="right_rear_wheel"
-    parent="base_link"
-    xyz="-0.23 -0.19 ${(-body_height/2.0)+(bearing_height/2.0)}" />
+  <xacro:pluto_wheel name="left_front_wheel" parent="virtual_axis_left">
+    <origin xyz="0.1075 0.095 0" rpy="0 0 0" />
+  </xacro:pluto_wheel>
+  <xacro:pluto_wheel name="left_middle_wheel" parent="virtual_axis_left">
+    <origin xyz="-0.1075 0.095 0" rpy="0 0 0 "/>
+  </xacro:pluto_wheel>
+  <xacro:pluto_wheel name="left_rear_wheel" parent="base_link">
+    <origin xyz="-0.23 0.19 ${(-body_height/2.0)+(bearing_height/2.0)}" rpy="0 0 0" />
+  </xacro:pluto_wheel>
+  <xacro:pluto_wheel name="right_front_wheel" parent="virtual_axis_right">
+    <origin xyz="0.1075 -0.095 0" rpy="0 0 0" />
+  </xacro:pluto_wheel>
+  <xacro:pluto_wheel name="right_middle_wheel" parent="virtual_axis_right">
+    <origin xyz="-0.1075 -0.095 0" rpy="0 0 0" />
+  </xacro:pluto_wheel>
+  <xacro:pluto_wheel name="right_rear_wheel" parent="base_link">
+    <origin xyz="-0.23 -0.19 ${(-body_height/2.0)+(bearing_height/2.0)}" rpy="0 0 0" />
+  </xacro:pluto_wheel>
   <link name="imu_center">
     <visual>
@@ -354,20 +314,4 @@
     </plugin>
   </gazebo>
-  <gazebo>
-    <plugin name="skid_steer_drive_controller" filename="libgazebo_ros_skid_steer_drive.so">
-      <updateRate>100.0</updateRate>
-      <robotNamespace>/</robotNamespace>
-      <leftFrontJoint>left_front_wheel_joint</leftFrontJoint>
-      <rightFrontJoint>right_front_wheel_joint</rightFrontJoint>
-      <leftRearJoint>left_rear_wheel_joint</leftRearJoint>
-      <rightRearJoint>right_rear_wheel_joint</rightRearJoint>
-      <wheelSeparation>${axis_length}</wheelSeparation>
-      <wheelDiameter>${2*wheel_radius}</wheelDiameter>
-      <robotBaseFrame>base_link</robotBaseFrame>
-      <torque>20</torque>
-      <topicName>cmd_vel</topicName>
-      <broadcastTF>false</broadcastTF>
-    </plugin>
-  </gazebo>
   <!-- publish ground truth for pose of base_footprint -->
   <gazebo>
@@ -386,8 +330,8 @@
       <type>transmission_interface/SimpleTransmission</type>
       <joint name="${name}_joint">
-        <hardwareInterface>EffortJointInterface</hardwareInterface>
+        <hardwareInterface>hardware_interface/EffortJointInterface</hardwareInterface>
       </joint>
       <actuator name="${name}_motor">
-        <hardwareInterface>EffortJointInterface</hardwareInterface>
+        <hardwareInterface>hardware_interface/EffortJointInterface</hardwareInterface>
         <mechanicalReduction>1</mechanicalReduction>
       </actuator>
@@ -396,3 +340,7 @@
   <xacro:simple_transmission name="virtual_left_to_base" />
   <xacro:simple_transmission name="virtual_right_to_base" />
+  <gazebo>
+    <plugin name="gazebo_ros_control" filename="libgazebo_ros_control.so">
+    </plugin>
+  </gazebo>
 </robot>
